Commit message: change mid70 color to aqua
Signed-off-by: Daisuke Sato <daisukes@cmu.edu>

File: urdf/mid70.xacro (robot description, xacro)
@@ -26,4 +26,7 @@
             <box size="${length} ${width} ${height}"/>
         </geometry>
+        <material name="aqua">
+          <color rgba="0.31 0.77 0.83 1" />
+        </material>
   </visual>
 </link>

Commit message: refactoring code, make downsample as xacro parameter
Signed-off-by: Daisuke Sato <daisukes@cmu.edu>

File: urdf/mid70.xacro (robot description, xacro)
@@ -1,38 +1,40 @@
 <?xml version="1.0" encoding="UTF-8"?>
 <robot xmlns:xacro="http://ros.org/wiki/xacro">
-  <xacro:property name="M_PI" value="3.14159"/>
-  <xacro:property name="laser_min_range" value="0.1"/>
-  <xacro:property name="laser_max_range" value="200.0"/>
-  <xacro:property name="horizontal_fov" value="70.4"/>
-  <xacro:property name="vertical_fov" value="70.4"/>
-  <xacro:property name="samples" value="10000"/>
-  <xacro:property name="resolution" value="0.002"/>
-<xacro:property name="mass" value="0.4" />
-<xacro:property name="length" value="0.1" />
-<xacro:property name="width" value="0.06" />
-<xacro:property name="height" value="0.06" />
+  <xacro:property name="M_PI" value="3.14159" />
+  <xacro:property name="laser_min_range" value="0.1" />
+  <xacro:property name="laser_max_range" value="200.0" />
+  <xacro:property name="horizontal_fov" value="70.4" />
+  <xacro:property name="vertical_fov" value="70.4" />
+  <xacro:property name="samples" value="10000" />
+  <xacro:property name="downsample" value="1" />
+  <xacro:property name="resolution" value="0.002" />
+  <xacro:property name="mass" value="0.4" />
+  <xacro:property name="length" value="0.1" />
+  <xacro:property name="width" value="0.06" />
+  <xacro:property name="height" value="0.06" />
   <xacro:macro name="box_inertia" params="m w h d">
     <inertial>
-      <origin xyz="0 0 0" rpy="${pi/2} 0 ${pi/2}"/>
-      <mass value="${m}"/>
-      <inertia ixx="${(m/12) * (h*h + d*d)}" ixy="0.0" ixz="0.0" iyy="${(m/12) * (w*w + d*d)}" iyz="0.0" izz="${(m/12) * (w*w + h*h)}"/>
+      <origin xyz="0 0 0" rpy="${pi/2} 0 ${pi/2}" />
+      <mass value="${m}" />
+      <inertia ixx="${(m/12) * (h*h + d*d)}" ixy="0.0" ixz="0.0" iyy="${(m/12) * (w*w + d*d)}"
+        iyz="0.0" izz="${(m/12) * (w*w + h*h)}" />
     </inertial>
   </xacro:macro>
   <xacro:macro name="mid70" params="name:='' parent:= 'base_link' topic:='mid70' *origin ">
-<link name="${name}">
-<xacro:box_inertia m="${length}" w="${width}" d="${length}" h="${height}"/>
-  <visual>
+    <link name="${name}">
+      <xacro:box_inertia m="${length}" w="${width}" d="${length}" h="${height}" />
+      <visual>
         <geometry>
-            <box size="${length} ${width} ${height}"/>
+          <box size="${length} ${width} ${height}" />
         </geometry>
         <material name="aqua">
           <color rgba="0.31 0.77 0.83 1" />
         </material>
-  </visual>
-</link>
+      </visual>
+    </link>
     <joint name="${name}_joint" type="fixed">
-      <parent link="${parent}"/>
-      <child link="${name}"/>
-      <xacro:insert_block name="origin"/>
+      <parent link="${parent}" />
+      <child link="${name}" />
+      <xacro:insert_block name="origin" />
     </joint>
     <gazebo reference="${name}">
@@ -41,61 +43,37 @@
         <visualize>false</visualize>
         <update_rate>10</update_rate>
-			<ray>
-			  <scan>
-				<horizontal>
-				<samples>${samples}</samples>
-				<resolution>1</resolution>
-				<min_angle>${-horizontal_fov/360*M_PI}</min_angle>
-				<max_angle>${horizontal_fov/360*M_PI}</max_angle>
-				</horizontal>
-				<vertical>
-				<samples>1</samples>
-				<resolution>1</resolution>
-				<min_angle>${-vertical_fov/360*M_PI}</min_angle>
-				<max_angle>${vertical_fov/360*M_PI}</max_angle>
-				</vertical>
-			  </scan>
-			  <range>
-				<min>${laser_min_range}</min>
-				<max>${laser_max_range}</max>
-				<resolution>0.002</resolution>
-			  </range>
-			  <noise>
-				<type>gaussian</type>
-				<mean>0.0</mean>
-				<stddev>0.01</stddev>
-			  </noise>
-			</ray>
+        <ray>
+          <scan>
+            <horizontal>
+              <samples>${samples}</samples>
+              <resolution>1</resolution>
+              <min_angle>${-horizontal_fov/360*M_PI}</min_angle>
+              <max_angle>${horizontal_fov/360*M_PI}</max_angle>
+            </horizontal>
+            <vertical>
+              <samples>1</samples>
+              <resolution>1</resolution>
+              <min_angle>${-vertical_fov/360*M_PI}</min_angle>
+              <max_angle>${vertical_fov/360*M_PI}</max_angle>
+            </vertical>
+          </scan>
+          <range>
+            <min>${laser_min_range}</min>
+            <max>${laser_max_range}</max>
+            <resolution>0.002</resolution>
+          </range>
+          <noise>
+            <type>gaussian</type>
+            <mean>0.0</mean>
+            <stddev>0.01</stddev>
+          </noise>
+        </ray>
         <plugin name="${name}_plugin" filename="libros2_livox.so">
-			<ray>
-			  <scan>
-				<horizontal>
-				<samples>${samples}</samples>
-				<resolution>1</resolution>
-				<min_angle>${-horizontal_fov/360*M_PI}</min_angle>
-				<max_angle>${horizontal_fov/360*M_PI}</max_angle>
-				</horizontal>
-				<vertical>
-				<samples>1</samples>
-				<resolution>1</resolution>
-				<min_angle>${-vertical_fov/360*M_PI}</min_angle>
-				<max_angle>${vertical_fov/360*M_PI}</max_angle>
-				</vertical>
-			  </scan>
-			  <range>
-				<min>${laser_min_range}</min>
-				<max>${laser_max_range}</max>
-				<resolution>0.002</resolution>
-			  </range>
-			  <noise>
-				<type>gaussian</type>
-				<mean>0.0</mean>
-				<stddev>0.01</stddev>
-			  </noise>
-			</ray>
-		  <samples>${samples}</samples>
-		  <downsample>1</downsample>
-		  <csv_file_name>$(find ros2_livox_simulation)/scan_mode/mid70.csv</csv_file_name>
-		  <topic>${topic}</topic>
+          <samples>${samples}</samples>
+          <downsample>${downsample}</downsample>
+          <min_range>${laser_min_range}</min_range>
+          <max_range>${laser_max_range}</max_range>
+          <csv_file_name>$(find ros2_livox_simulation)/scan_mode/mid70.csv</csv_file_name>
+          <topic>${topic}</topic>
         </plugin>
       </sensor>

Commit message: implemented GPU by using grid approximation
Signed-off-by: Daisuke Sato <daisukes@cmu.edu>

File: urdf/mid70.xacro (robot description, xacro)
@@ -7,4 +7,5 @@
   <xacro:property name="vertical_fov" value="70.4" />
   <xacro:property name="samples" value="10000" />
+  <xacro:property name="gpu_samples" value="512" />
   <xacro:property name="downsample" value="1" />
   <xacro:property name="resolution" value="0.002" />
@@ -21,5 +22,5 @@
     </inertial>
   </xacro:macro>
-  <xacro:macro name="mid70" params="name:='' parent:= 'base_link' topic:='mid70' *origin ">
+  <xacro:macro name="mid70" params="name:='' parent:= 'base_link' topic:='mid70' *origin gpu:=true">
     <link name="${name}">
       <xacro:box_inertia m="${length}" w="${width}" d="${length}" h="${height}" />
@@ -39,43 +40,87 @@
     </joint>
     <gazebo reference="${name}">
-      <sensor type="ray" name="${name}">
-        <pose>0 0 0 0 0 0</pose>
-        <visualize>false</visualize>
-        <update_rate>10</update_rate>
-        <ray>
-          <scan>
-            <horizontal>
-              <samples>${samples}</samples>
-              <resolution>1</resolution>
-              <min_angle>${-horizontal_fov/360*M_PI}</min_angle>
-              <max_angle>${horizontal_fov/360*M_PI}</max_angle>
-            </horizontal>
-            <vertical>
-              <samples>1</samples>
-              <resolution>1</resolution>
-              <min_angle>${-vertical_fov/360*M_PI}</min_angle>
-              <max_angle>${vertical_fov/360*M_PI}</max_angle>
-            </vertical>
-          </scan>
-          <range>
-            <min>${laser_min_range}</min>
-            <max>${laser_max_range}</max>
-            <resolution>0.002</resolution>
-          </range>
-          <noise>
-            <type>gaussian</type>
-            <mean>0.0</mean>
-            <stddev>0.01</stddev>
-          </noise>
-        </ray>
-        <plugin name="${name}_plugin" filename="libros2_livox.so">
-          <samples>${samples}</samples>
-          <downsample>${downsample}</downsample>
-          <min_range>${laser_min_range}</min_range>
-          <max_range>${laser_max_range}</max_range>
-          <csv_file_name>$(find ros2_livox_simulation)/scan_mode/mid70.csv</csv_file_name>
-          <topic>${topic}</topic>
-        </plugin>
-      </sensor>
+      <xacro:if value="${gpu}">
+        <sensor type="gpu_ray" name="${name}">
+          <pose>0 0 0 0 0 0</pose>
+          <visualize>false</visualize>
+          <update_rate>10</update_rate>
+          <ray>
+            <scan>
+              <horizontal>
+                <samples>${gpu_samples}</samples>
+                <resolution>1</resolution>
+                <min_angle>${-horizontal_fov/360*M_PI}</min_angle>
+                <max_angle>${horizontal_fov/360*M_PI}</max_angle>
+              </horizontal>
+              <vertical>
+                <samples>${gpu_samples}</samples>
+                <resolution>1</resolution>
+                <min_angle>${-vertical_fov/360*M_PI}</min_angle>
+                <max_angle>${vertical_fov/360*M_PI}</max_angle>
+              </vertical>
+            </scan>
+            <range>
+              <min>${laser_min_range}</min>
+              <max>${laser_max_range}</max>
+              <resolution>0.002</resolution>
+            </range>
+            <noise>
+              <type>gaussian</type>
+              <mean>0.0</mean>
+              <stddev>0.01</stddev>
+            </noise>
+          </ray>
+          <plugin name="${name}_plugin" filename="libros2_livox.so">
+            <samples>${samples}</samples>
+            <grid>${gpu_samples}</grid>
+            <downsample>${downsample}</downsample>
+            <min_range>${laser_min_range}</min_range>
+            <max_range>${laser_max_range}</max_range>
+            <csv_file_name>$(find ros2_livox_simulation)/scan_mode/mid70.csv</csv_file_name>
+            <topic>${topic}</topic>
+          </plugin>
+        </sensor>
+      </xacro:if>
+      <xacro:unless value="${gpu}">
+        <sensor type="ray" name="${name}">
+          <pose>0 0 0 0 0 0</pose>
+          <visualize>false</visualize>
+          <update_rate>10</update_rate>
+          <ray>
+            <scan>
+              <horizontal>
+                <samples>${samples}</samples>
+                <resolution>1</resolution>
+                <min_angle>${-horizontal_fov/360*M_PI}</min_angle>
+                <max_angle>${horizontal_fov/360*M_PI}</max_angle>
+              </horizontal>
+              <vertical>
+                <samples>1</samples>
+                <resolution>1</resolution>
+                <min_angle>${-vertical_fov/360*M_PI}</min_angle>
+                <max_angle>${vertical_fov/360*M_PI}</max_angle>
+              </vertical>
+            </scan>
+            <range>
+              <min>${laser_min_range}</min>
+              <max>${laser_max_range}</max>
+              <resolution>0.002</resolution>
+            </range>
+            <noise>
+              <type>gaussian</type>
+              <mean>0.0</mean>
+              <stddev>0.01</stddev>
+            </noise>
+          </ray>
+          <plugin name="${name}_plugin" filename="libros2_livox.so">
+            <samples>${samples}</samples>
+            <downsample>${downsample}</downsample>
+            <min_range>${laser_min_range}</min_range>
+            <max_range>${laser_max_range}</max_range>
+            <csv_file_name>$(find ros2_livox_simulation)/scan_mode/mid70.csv</csv_file_name>
+            <topic>${topic}</topic>
+          </plugin>
+        </sensor>
+      </xacro:unless>
     </gazebo>
   </xacro:macro>

Commit message: add gpu interpolation
Signed-off-by: Daisuke Sato <daisukes@cmu.edu>

File: urdf/mid70.xacro (robot description, xacro)
@@ -22,5 +22,5 @@
     </inertial>
   </xacro:macro>
-  <xacro:macro name="mid70" params="name:='' parent:= 'base_link' topic:='mid70' *origin gpu:=true">
+  <xacro:macro name="mid70" params="name:='' parent:= 'base_link' topic:='mid70' *origin gpu:=true interpolation:=true">
     <link name="${name}">
       <xacro:box_inertia m="${length}" w="${width}" d="${length}" h="${height}" />
@@ -74,4 +74,5 @@
             <samples>${samples}</samples>
             <grid>${gpu_samples}</grid>
+            <interpolation>${interpolation}</interpolation>
             <downsample>${downsample}</downsample>
             <min_range>${laser_min_range}</min_range>
